Commit message: Add AI Sapiens Phase 2 stack

File: ai_sapiens_description/urdf/k1_rev1/k1.urdf (robot description, URDF)
Before this commit: robot k1, 25 links, 24 joints
Links:
- link head_link: mass 5.502976800e-01 -> 7.279675100e-01
- link left_ankle_roll_link: geometry collision sphere radius=0.005; collision sphere radius=0.005
- link right_ankle_roll_link: geometry collision sphere radius=0.005; collision sphere radius=0.005
Joints:
- joint head_joint: origin xyz=-0.0185 0 0.385 rpy=0 0 0 -> xyz=-0.02725 0 0.361 rpy=0 0 0
