Commit message: Add MujocoSystem ros2_control plugin and sim_mujoco xacro wiring
Signed-off-by: Kiwoong Park <abrahamola80@gmail.com>

File: ai_sapiens_description/ros2_control/k1_rev1/k1.ros2_control.xacro (robot description, xacro)
@@ -7,25 +7,31 @@
   <xacro:include filename="$(find ai_sapiens_description)/ros2_control/k1_rev1/k1_imu.ros2_control.xacro" />
   <xacro:include filename="$(find ai_sapiens_description)/ros2_control/k1_rev1/k1_hat.ros2_control.xacro" />
+  <xacro:include filename="$(find ai_sapiens_description)/ros2_control/k1_rev1/k1_mujoco.ros2_control.xacro" />
   <xacro:property name="default_use_mock_hardware" value="false" />
   <xacro:property name="default_mock_sensor_commands" value="false" />
-  <xacro:macro name="k1_system" params="use_mock_hardware:=^|${default_use_mock_hardware} mock_sensor_commands:=^|${default_mock_sensor_commands}">
-    <xacro:k1_right_arm_system
-      use_mock_hardware="${use_mock_hardware}"
-      mock_sensor_commands="${mock_sensor_commands}" />
-    <xacro:k1_left_arm_system
-      use_mock_hardware="${use_mock_hardware}"
-      mock_sensor_commands="${mock_sensor_commands}" />
-    <xacro:k1_left_leg_system
-      use_mock_hardware="${use_mock_hardware}"
-      mock_sensor_commands="${mock_sensor_commands}" />
-    <xacro:k1_right_leg_system
-      use_mock_hardware="${use_mock_hardware}"
-      mock_sensor_commands="${mock_sensor_commands}" />
-    <xacro:k1_imu_system
-      use_mock_hardware="${use_mock_hardware}"
-      mock_sensor_commands="${mock_sensor_commands}" />
-    <xacro:k1_hat_system
-      use_mock_hardware="${use_mock_hardware}"
-      mock_sensor_commands="${mock_sensor_commands}" />
+  <xacro:macro name="k1_system" params="use_mock_hardware:=^|${default_use_mock_hardware} mock_sensor_commands:=^|${default_mock_sensor_commands} sim_mujoco:=^|false mujoco_viewer:=^|true mujoco_gantry:=^|true">
+    <xacro:if value="${sim_mujoco}">
+      <xacro:k1_mujoco_system viewer="${mujoco_viewer}" gantry="${mujoco_gantry}"/>
+    </xacro:if>
+    <xacro:unless value="${sim_mujoco}">
+      <xacro:k1_right_arm_system
+        use_mock_hardware="${use_mock_hardware}"
+        mock_sensor_commands="${mock_sensor_commands}" />
+      <xacro:k1_left_arm_system
+        use_mock_hardware="${use_mock_hardware}"
+        mock_sensor_commands="${mock_sensor_commands}" />
+      <xacro:k1_left_leg_system
+        use_mock_hardware="${use_mock_hardware}"
+        mock_sensor_commands="${mock_sensor_commands}" />
+      <xacro:k1_right_leg_system
+        use_mock_hardware="${use_mock_hardware}"
+        mock_sensor_commands="${mock_sensor_commands}" />
+      <xacro:k1_imu_system
+        use_mock_hardware="${use_mock_hardware}"
+        mock_sensor_commands="${mock_sensor_commands}" />
+      <xacro:k1_hat_system
+        use_mock_hardware="${use_mock_hardware}"
+        mock_sensor_commands="${mock_sensor_commands}" />
+    </xacro:unless>
   </xacro:macro>
 </robot>

File: ai_sapiens_description/urdf/k1_rev1/k1.urdf.xacro (robot description, xacro)
@@ -6,4 +6,7 @@
   <xacro:arg name="prefix" default="" />
   <xacro:arg name="model" default="k1_rev1" />
+  <xacro:arg name="sim_mujoco" default="false" />
+  <xacro:arg name="mujoco_viewer" default="true" />
+  <xacro:arg name="mujoco_gantry" default="true" />
   <xacro:include filename="$(find ai_sapiens_description)/urdf/k1_rev1/$(arg model).urdf.xacro" />
   <xacro:include filename="$(find ai_sapiens_description)/ros2_control/k1_rev1/k1.ros2_control.xacro" />
@@ -11,4 +14,7 @@
   <xacro:k1_system
     use_mock_hardware="$(arg use_mock_hardware)"
-    mock_sensor_commands="$(arg mock_sensor_commands)"/>
+    mock_sensor_commands="$(arg mock_sensor_commands)"
+    sim_mujoco="$(arg sim_mujoco)"
+    mujoco_viewer="$(arg mujoco_viewer)"
+    mujoco_gantry="$(arg mujoco_gantry)"/>
 </robot>

Commit message: Wire RadioMaster USB into K1 ros2_control

File: ai_sapiens_description/ros2_control/k1_rev1/k1.ros2_control.xacro (robot description, xacro)
@@ -7,7 +7,8 @@
   <xacro:include filename="$(find ai_sapiens_description)/ros2_control/k1_rev1/k1_imu.ros2_control.xacro" />
   <xacro:include filename="$(find ai_sapiens_description)/ros2_control/k1_rev1/k1_hat.ros2_control.xacro" />
+  <xacro:include filename="$(find ai_sapiens_description)/ros2_control/k1_rev1/k1_radiomaster_pocket_usb.ros2_control.xacro" />
   <xacro:property name="default_use_mock_hardware" value="false" />
   <xacro:property name="default_mock_sensor_commands" value="false" />
-  <xacro:macro name="k1_system" params="use_mock_hardware:=^|${default_use_mock_hardware} mock_sensor_commands:=^|${default_mock_sensor_commands}">
+  <xacro:macro name="k1_system" params="use_mock_hardware:=^|${default_use_mock_hardware} mock_sensor_commands:=^|${default_mock_sensor_commands} radiomaster_pocket_usb:=^|false radiomaster_pocket_usb_device:=^|/dev/input/js0">
     <xacro:k1_right_arm_system
       use_mock_hardware="${use_mock_hardware}"
@@ -25,7 +26,12 @@
       use_mock_hardware="${use_mock_hardware}"
       mock_sensor_commands="${mock_sensor_commands}" />
-    <xacro:k1_hat_system
-      use_mock_hardware="${use_mock_hardware}"
-      mock_sensor_commands="${mock_sensor_commands}" />
+    <xacro:if value="${radiomaster_pocket_usb}">
+      <xacro:k1_radiomaster_pocket_usb_system device="${radiomaster_pocket_usb_device}" />
+    </xacro:if>
+    <xacro:unless value="${radiomaster_pocket_usb}">
+      <xacro:k1_hat_system
+        use_mock_hardware="${use_mock_hardware}"
+        mock_sensor_commands="${mock_sensor_commands}" />
+    </xacro:unless>
   </xacro:macro>
 </robot>

File: ai_sapiens_description/urdf/k1_rev1/k1.urdf.xacro (robot description, xacro)
@@ -6,4 +6,6 @@
   <xacro:arg name="prefix" default="" />
   <xacro:arg name="model" default="k1_rev1" />
+  <xacro:arg name="radiomaster_pocket_usb" default="false" />
+  <xacro:arg name="radiomaster_pocket_usb_device" default="/dev/input/js0" />
   <xacro:include filename="$(find ai_sapiens_description)/urdf/k1_rev1/$(arg model).urdf.xacro" />
   <xacro:include filename="$(find ai_sapiens_description)/ros2_control/k1_rev1/k1.ros2_control.xacro" />
@@ -11,4 +13,6 @@
   <xacro:k1_system
     use_mock_hardware="$(arg use_mock_hardware)"
-    mock_sensor_commands="$(arg mock_sensor_commands)"/>
+    mock_sensor_commands="$(arg mock_sensor_commands)"
+    radiomaster_pocket_usb="$(arg radiomaster_pocket_usb)"
+    radiomaster_pocket_usb_device="$(arg radiomaster_pocket_usb_device)"/>
 </robot>

Commit message: Separate real and MuJoCo ros2_control definitions
Signed-off-by: Kiwoong Park <abrahamola80@gmail.com>

File: ai_sapiens_description/ros2_control/k1_rev1/k1.ros2_control.xacro (robot description, xacro)
@@ -7,31 +7,25 @@
   <xacro:include filename="$(find ai_sapiens_description)/ros2_control/k1_rev1/k1_imu.ros2_control.xacro" />
   <xacro:include filename="$(find ai_sapiens_description)/ros2_control/k1_rev1/k1_hat.ros2_control.xacro" />
-  <xacro:include filename="$(find ai_sapiens_description)/ros2_control/k1_rev1/k1_mujoco.ros2_control.xacro" />
   <xacro:property name="default_use_mock_hardware" value="false" />
   <xacro:property name="default_mock_sensor_commands" value="false" />
-  <xacro:macro name="k1_system" params="use_mock_hardware:=^|${default_use_mock_hardware} mock_sensor_commands:=^|${default_mock_sensor_commands} sim_mujoco:=^|false mujoco_viewer:=^|true mujoco_gantry:=^|true">
-    <xacro:if value="${sim_mujoco}">
-      <xacro:k1_mujoco_system viewer="${mujoco_viewer}" gantry="${mujoco_gantry}"/>
-    </xacro:if>
-    <xacro:unless value="${sim_mujoco}">
-      <xacro:k1_right_arm_system
-        use_mock_hardware="${use_mock_hardware}"
-        mock_sensor_commands="${mock_sensor_commands}" />
-      <xacro:k1_left_arm_system
-        use_mock_hardware="${use_mock_hardware}"
-        mock_sensor_commands="${mock_sensor_commands}" />
-      <xacro:k1_left_leg_system
-        use_mock_hardware="${use_mock_hardware}"
-        mock_sensor_commands="${mock_sensor_commands}" />
-      <xacro:k1_right_leg_system
-        use_mock_hardware="${use_mock_hardware}"
-        mock_sensor_commands="${mock_sensor_commands}" />
-      <xacro:k1_imu_system
-        use_mock_hardware="${use_mock_hardware}"
-        mock_sensor_commands="${mock_sensor_commands}" />
-      <xacro:k1_hat_system
-        use_mock_hardware="${use_mock_hardware}"
-        mock_sensor_commands="${mock_sensor_commands}" />
-    </xacro:unless>
+  <xacro:macro name="k1_system" params="use_mock_hardware:=^|${default_use_mock_hardware} mock_sensor_commands:=^|${default_mock_sensor_commands}">
+    <xacro:k1_right_arm_system
+      use_mock_hardware="${use_mock_hardware}"
+      mock_sensor_commands="${mock_sensor_commands}" />
+    <xacro:k1_left_arm_system
+      use_mock_hardware="${use_mock_hardware}"
+      mock_sensor_commands="${mock_sensor_commands}" />
+    <xacro:k1_left_leg_system
+      use_mock_hardware="${use_mock_hardware}"
+      mock_sensor_commands="${mock_sensor_commands}" />
+    <xacro:k1_right_leg_system
+      use_mock_hardware="${use_mock_hardware}"
+      mock_sensor_commands="${mock_sensor_commands}" />
+    <xacro:k1_imu_system
+      use_mock_hardware="${use_mock_hardware}"
+      mock_sensor_commands="${mock_sensor_commands}" />
+    <xacro:k1_hat_system
+      use_mock_hardware="${use_mock_hardware}"
+      mock_sensor_commands="${mock_sensor_commands}" />
   </xacro:macro>
 </robot>

File: ai_sapiens_description/urdf/k1_rev1/k1.urdf.xacro (robot description, xacro)
@@ -11,10 +11,15 @@
   <xacro:include filename="$(find ai_sapiens_description)/urdf/k1_rev1/$(arg model).urdf.xacro" />
   <xacro:include filename="$(find ai_sapiens_description)/ros2_control/k1_rev1/k1.ros2_control.xacro" />
+  <xacro:include filename="$(find ai_sapiens_description)/ros2_control/k1_rev1/k1_mujoco.ros2_control.xacro" />
   <xacro:k1/>
-  <xacro:k1_system
-    use_mock_hardware="$(arg use_mock_hardware)"
-    mock_sensor_commands="$(arg mock_sensor_commands)"
-    sim_mujoco="$(arg sim_mujoco)"
-    mujoco_viewer="$(arg mujoco_viewer)"
-    mujoco_gantry="$(arg mujoco_gantry)"/>
+  <xacro:if value="$(arg sim_mujoco)">
+    <xacro:k1_mujoco_system
+      viewer="$(arg mujoco_viewer)"
+      gantry="$(arg mujoco_gantry)"/>
+  </xacro:if>
+  <xacro:unless value="$(arg sim_mujoco)">
+    <xacro:k1_system
+      use_mock_hardware="$(arg use_mock_hardware)"
+      mock_sensor_commands="$(arg mock_sensor_commands)"/>
+  </xacro:unless>
 </robot>

Commit message: Wire RadioMaster USB into MuJoCo bringup
Signed-off-by: Kiwoong Park <abrahamola80@gmail.com>

File: ai_sapiens_description/ros2_control/k1_rev1/k1.ros2_control.xacro (robot description, xacro)
@@ -7,8 +7,7 @@
   <xacro:include filename="$(find ai_sapiens_description)/ros2_control/k1_rev1/k1_imu.ros2_control.xacro" />
   <xacro:include filename="$(find ai_sapiens_description)/ros2_control/k1_rev1/k1_hat.ros2_control.xacro" />
-  <xacro:include filename="$(find ai_sapiens_description)/ros2_control/k1_rev1/k1_radiomaster_pocket_usb.ros2_control.xacro" />
   <xacro:property name="default_use_mock_hardware" value="false" />
   <xacro:property name="default_mock_sensor_commands" value="false" />
-  <xacro:macro name="k1_system" params="use_mock_hardware:=^|${default_use_mock_hardware} mock_sensor_commands:=^|${default_mock_sensor_commands} radiomaster_pocket_usb:=^|false radiomaster_pocket_usb_device:=^|/dev/input/js0">
+  <xacro:macro name="k1_system" params="use_mock_hardware:=^|${default_use_mock_hardware} mock_sensor_commands:=^|${default_mock_sensor_commands}">
     <xacro:k1_right_arm_system
       use_mock_hardware="${use_mock_hardware}"
@@ -26,12 +25,7 @@
       use_mock_hardware="${use_mock_hardware}"
       mock_sensor_commands="${mock_sensor_commands}" />
-    <xacro:if value="${radiomaster_pocket_usb}">
-      <xacro:k1_radiomaster_pocket_usb_system device="${radiomaster_pocket_usb_device}" />
-    </xacro:if>
-    <xacro:unless value="${radiomaster_pocket_usb}">
-      <xacro:k1_hat_system
-        use_mock_hardware="${use_mock_hardware}"
-        mock_sensor_commands="${mock_sensor_commands}" />
-    </xacro:unless>
+    <xacro:k1_hat_system
+      use_mock_hardware="${use_mock_hardware}"
+      mock_sensor_commands="${mock_sensor_commands}" />
   </xacro:macro>
 </robot>

File: ai_sapiens_description/ros2_control/k1_rev1/k1_mujoco.ros2_control.xacro (robot description, xacro)
@@ -1,5 +1,7 @@
 <?xml version="1.0"?>
 <robot xmlns:xacro="http://www.ros.org/wiki/xacro">
-  <xacro:macro name="k1_mujoco_system" params="viewer:=^|true gantry:=^|true">
+  <xacro:macro
+    name="k1_mujoco_system"
+    params="viewer:=^|true gantry:=^|true external_hat:=^|false">
     <ros2_control name="k1_mujoco" type="system">
       <hardware>
@@ -62,35 +64,37 @@
         <state_interface name="orientation.z"/>
       </sensor>
-      <sensor name="hat">
-        <state_interface name="Hardware Error Status"/>
-        <state_interface name="Realtime Tick"/>
-        <state_interface name="E-stop Active"/>
-        <state_interface name="BMS SOC"/>
-        <state_interface name="BMS Voltage"/>
-        <state_interface name="BMS Current"/>
-        <state_interface name="BMS Temperature"/>
-        <state_interface name="BMS Service Error Flags"/>
-        <state_interface name="BMS Remaining Energy"/>
-        <state_interface name="CRSF Failsafe"/>
-        <state_interface name="CRSF Link Quality"/>
-        <state_interface name="CRSF RSSI 1"/>
-        <state_interface name="CRSF Last Frame Age"/>
-        <state_interface name="RC Channel 1"/>
-        <state_interface name="RC Channel 2"/>
-        <state_interface name="RC Channel 3"/>
-        <state_interface name="RC Channel 4"/>
-        <state_interface name="RC Channel 5"/>
-        <state_interface name="RC Channel 6"/>
-        <state_interface name="RC Channel 7"/>
-        <state_interface name="RC Channel 8"/>
-        <state_interface name="RC Channel 9"/>
-        <state_interface name="RC Channel 10"/>
-        <state_interface name="RC Channel 11"/>
-        <state_interface name="RC Channel 12"/>
-        <state_interface name="RC Channel 13"/>
-        <state_interface name="RC Channel 14"/>
-        <state_interface name="RC Channel 15"/>
-        <state_interface name="RC Channel 16"/>
-      </sensor>
+      <xacro:unless value="${external_hat}">
+        <sensor name="hat">
+          <state_interface name="Hardware Error Status"/>
+          <state_interface name="Realtime Tick"/>
+          <state_interface name="E-stop Active"/>
+          <state_interface name="BMS SOC"/>
+          <state_interface name="BMS Voltage"/>
+          <state_interface name="BMS Current"/>
+          <state_interface name="BMS Temperature"/>
+          <state_interface name="BMS Service Error Flags"/>
+          <state_interface name="BMS Remaining Energy"/>
+          <state_interface name="CRSF Failsafe"/>
+          <state_interface name="CRSF Link Quality"/>
+          <state_interface name="CRSF RSSI 1"/>
+          <state_interface name="CRSF Last Frame Age"/>
+          <state_interface name="RC Channel 1"/>
+          <state_interface name="RC Channel 2"/>
+          <state_interface name="RC Channel 3"/>
+          <state_interface name="RC Channel 4"/>
+          <state_interface name="RC Channel 5"/>
+          <state_interface name="RC Channel 6"/>
+          <state_interface name="RC Channel 7"/>
+          <state_interface name="RC Channel 8"/>
+          <state_interface name="RC Channel 9"/>
+          <state_interface name="RC Channel 10"/>
+          <state_interface name="RC Channel 11"/>
+          <state_interface name="RC Channel 12"/>
+          <state_interface name="RC Channel 13"/>
+          <state_interface name="RC Channel 14"/>
+          <state_interface name="RC Channel 15"/>
+          <state_interface name="RC Channel 16"/>
+        </sensor>
+      </xacro:unless>
     </ros2_control>
   </xacro:macro>

File: ai_sapiens_description/ros2_control/k1_rev1/k1_radiomaster_usb.ros2_control.xacro (robot description, xacro)
@@ -1,8 +1,8 @@
 <?xml version="1.0"?>
 <robot xmlns:xacro="http://www.ros.org/wiki/xacro">
-  <xacro:macro name="k1_radiomaster_pocket_usb_system" params="device:=^|/dev/input/js0">
-    <ros2_control name="k1_radiomaster_pocket_usb" type="sensor" rw_rate="100">
+  <xacro:macro name="k1_radiomaster_usb_system" params="device:=^|/dev/input/js0">
+    <ros2_control name="k1_radiomaster_usb" type="sensor" rw_rate="100">
       <hardware>
-        <plugin>radiomaster_pocket_usb_hardware_interface/RadiomasterPocketUsbHardwareInterface</plugin>
+        <plugin>radiomaster_usb_hardware_interface/RadiomasterUsbHardwareInterface</plugin>
         <param name="device">${device}</param>
         <param name="reconnect_interval_ms">1000.0</param>

File: ai_sapiens_description/urdf/k1_rev1/k1.urdf.xacro (robot description, xacro)
@@ -9,21 +9,25 @@
   <xacro:arg name="mujoco_viewer" default="true" />
   <xacro:arg name="mujoco_gantry" default="true" />
-  <xacro:arg name="radiomaster_pocket_usb" default="false" />
-  <xacro:arg name="radiomaster_pocket_usb_device" default="/dev/input/js0" />
+  <xacro:arg name="radiomaster_usb" default="false" />
+  <xacro:arg name="radiomaster_usb_device" default="/dev/input/js0" />
   <xacro:include filename="$(find ai_sapiens_description)/urdf/k1_rev1/$(arg model).urdf.xacro" />
   <xacro:include filename="$(find ai_sapiens_description)/ros2_control/k1_rev1/k1.ros2_control.xacro" />
   <xacro:include filename="$(find ai_sapiens_description)/ros2_control/k1_rev1/k1_mujoco.ros2_control.xacro" />
+  <xacro:include filename="$(find ai_sapiens_description)/ros2_control/k1_rev1/k1_radiomaster_usb.ros2_control.xacro" />
   <xacro:k1/>
   <xacro:if value="$(arg sim_mujoco)">
     <xacro:k1_mujoco_system
       viewer="$(arg mujoco_viewer)"
-      gantry="$(arg mujoco_gantry)"/>
+      gantry="$(arg mujoco_gantry)"
+      external_hat="$(arg radiomaster_usb)"/>
+    <xacro:if value="$(arg radiomaster_usb)">
+      <xacro:k1_radiomaster_usb_system
+        device="$(arg radiomaster_usb_device)"/>
+    </xacro:if>
   </xacro:if>
   <xacro:unless value="$(arg sim_mujoco)">
     <xacro:k1_system
       use_mock_hardware="$(arg use_mock_hardware)"
-      mock_sensor_commands="$(arg mock_sensor_commands)"
-      radiomaster_pocket_usb="$(arg radiomaster_pocket_usb)"
-      radiomaster_pocket_usb_device="$(arg radiomaster_pocket_usb_device)"/>
+      mock_sensor_commands="$(arg mock_sensor_commands)"/>
   </xacro:unless>
 </robot>
