Commit message: Add dual RadioMaster group control with individual override
Signed-off-by: Kiwoong Park <abrahamola80@gmail.com>

File: ai_sapiens_description/ros2_control/k1_rev1/k1_radiomaster_usb.ros2_control.xacro (robot description, xacro)
@@ -1,6 +1,6 @@
 <?xml version="1.0"?>
 <robot xmlns:xacro="http://www.ros.org/wiki/xacro">
-  <xacro:macro name="k1_radiomaster_usb_system" params="device:=^|/dev/input/js0">
-    <ros2_control name="k1_radiomaster_usb" type="sensor" rw_rate="100">
+  <xacro:macro name="k1_radiomaster_usb_system" params="device:=^|/dev/input/js0 name:=k1_radiomaster_usb sensor_name:=hat">
+    <ros2_control name="${name}" type="sensor" rw_rate="100">
       <hardware>
         <plugin>radiomaster_usb_hardware_interface/RadiomasterUsbHardwareInterface</plugin>
@@ -10,5 +10,5 @@
         <param name="rc_channel_defaults">1500,1500,1500,1500,1000,1500,1000,1000,1000,1000,1000,1000,1500,1500,1500,1500</param>
       </hardware>
-      <sensor name="hat">
+      <sensor name="${sensor_name}">
         <state_interface name="Hardware Error Status"/>
         <state_interface name="Realtime Tick"/>

File: ai_sapiens_description/urdf/k1_rev1/k1.urdf.xacro (robot description, xacro)
@@ -11,4 +11,6 @@
   <xacro:arg name="radiomaster_usb" default="false" />
   <xacro:arg name="radiomaster_usb_device" default="/dev/input/js0" />
+  <xacro:arg name="group_usb" default="false" />
+  <xacro:arg name="group_usb_device" default="/dev/input/js1" />
   <xacro:include filename="$(find ai_sapiens_description)/urdf/k1_rev1/$(arg model).urdf.xacro" />
   <xacro:include filename="$(find ai_sapiens_description)/ros2_control/k1_rev1/k1.ros2_control.xacro" />
@@ -24,4 +26,9 @@
         device="$(arg radiomaster_usb_device)"/>
     </xacro:if>
+    <xacro:if value="$(arg group_usb)">
+      <xacro:k1_radiomaster_usb_system
+        device="$(arg group_usb_device)"
+        name="k1_group_usb" sensor_name="group_hat"/>
+    </xacro:if>
   </xacro:if>
   <xacro:unless value="$(arg sim_mujoco)">

Commit message: Expose dual MuJoCo USB receivers through the shared HAT interface
Read the individual and optional group USB devices in one RadioMaster hardware
component. Export hat/RC Channel 1-16 and hat/Remote 2 CH1-16 so MuJoCo uses the
same broadcaster configuration as the real K1 HAT without duplicate state
interfaces. Keep the existing single-device configuration and launch flags.

Track USB connection, axis initialization, and reconnect state per receiver.
Preserve the individual receiver's existing shared status behavior and mark
unavailable group channels invalid so group USB loss does not invalidate the
individual input. The real firmware's per-receiver CRSF status remains outside
this change.

Validation: both packages build; five simulated joystick lifecycle/read tests
pass; description tests report eight passed and one skipped; RC broadcaster
regression tests pass. Real, dual-USB, and single-USB Xacro interfaces match the
common controller YAML. C++ formatting passes. The existing description
copyright check still fails because package-level LICENSE and CONTRIBUTING.md
are absent. Physical joystick and robot operation were not tested.

Signed-off-by: Kiwoong Park <abrahamola80@gmail.com>

File: ai_sapiens_description/ros2_control/k1_rev1/k1_radiomaster_usb.ros2_control.xacro (robot description, xacro)
@@ -1,7 +1,10 @@
 <?xml version="1.0"?>
 <robot xmlns:xacro="http://www.ros.org/wiki/xacro">
-  <xacro:macro name="k1_radiomaster_usb_system" params="device:=^|/dev/input/js0 name:=k1_radiomaster_usb sensor_name:=hat">
+  <xacro:macro name="k1_radiomaster_usb_system" params="device:=^|/dev/input/js0 name:=k1_radiomaster_usb sensor_name:=hat group_enabled:=false group_device:=/dev/input/js1">
     <ros2_control name="${name}" type="sensor" rw_rate="100">
       <hardware>
+        <xacro:if value="${group_enabled}">
+          <param name="group_device">${group_device}</param>
+        </xacro:if>
         <plugin>radiomaster_usb_hardware_interface/RadiomasterUsbHardwareInterface</plugin>
         <param name="device">${device}</param>
@@ -34,4 +37,22 @@
         <state_interface name="RC Channel 15"/>
         <state_interface name="RC Channel 16"/>
+        <xacro:if value="${group_enabled}">
+          <state_interface name="Remote 2 CH1"/>
+          <state_interface name="Remote 2 CH2"/>
+          <state_interface name="Remote 2 CH3"/>
+          <state_interface name="Remote 2 CH4"/>
+          <state_interface name="Remote 2 CH5"/>
+          <state_interface name="Remote 2 CH6"/>
+          <state_interface name="Remote 2 CH7"/>
+          <state_interface name="Remote 2 CH8"/>
+          <state_interface name="Remote 2 CH9"/>
+          <state_interface name="Remote 2 CH10"/>
+          <state_interface name="Remote 2 CH11"/>
+          <state_interface name="Remote 2 CH12"/>
+          <state_interface name="Remote 2 CH13"/>
+          <state_interface name="Remote 2 CH14"/>
+          <state_interface name="Remote 2 CH15"/>
+          <state_interface name="Remote 2 CH16"/>
+        </xacro:if>
       </sensor>
     </ros2_control>

File: ai_sapiens_description/urdf/k1_rev1/k1.urdf.xacro (robot description, xacro)
@@ -24,10 +24,7 @@
     <xacro:if value="$(arg radiomaster_usb)">
       <xacro:k1_radiomaster_usb_system
-        device="$(arg radiomaster_usb_device)"/>
-    </xacro:if>
-    <xacro:if value="$(arg group_usb)">
-      <xacro:k1_radiomaster_usb_system
-        device="$(arg group_usb_device)"
-        name="k1_group_usb" sensor_name="group_hat"/>
+        device="$(arg radiomaster_usb_device)"
+        group_enabled="$(arg group_usb)"
+        group_device="$(arg group_usb_device)"/>
     </xacro:if>
   </xacro:if>
